File: atreusAir.kicad_pcb (KiCad board)
At the start: 2 copper layers, 239 x 97 mm, 90 parts, among them SW1 POWER, SW10 Push, SW11 Push, SW12 Push, SW13 Push, SW14 Push, SW15 Push, SW16 Push, SW17 Push, SW18 Push, SW19 Push, SW2 Push, SW20 Push, SW21 Push, SW22 Push, SW23 Push, SW24 Push, SW25 Push, SW26 Push, SW27 Push, SW28 Push, SW29 Push, SW3 Push, SW30 Push, SW31 Push, SW32 Push, SW33 Push, SW34 Push, SW35 Push, SW36 Push, SW37 Push, SW38 Push, SW39 Push, SW4 Push, SW40 Push, SW41 Push, SW42 Push, SW43 Push, SW5 Push, SW6 Push, SW7 Push, SW8 Push, SW9 Push, U1 Feather_Bluefruit_LE

Commit message: switches sorted but not yet connected
Parts:
- D1, D10, D11, D12, D13, D14, D15, D16, D17, D18, D19, D2, D20, D21, D22, D23, D24, D25, D26, D27, D28, D29, D3, D30, D31, D32, D34, D35, D36, D37, D38, D39, D4, D40, D41, D42, D5, D6, D7, D8, D9, R2: moved to F.Cu
- D33: value D -> 18-225/R6G6C-A01/3T; footprint Diodes_SMD:D_0603 -> atreusAir:R6G6C-A01; moved to F.Cu
- D43: value 18-225/R6G6C-A01/3T -> D; footprint atreusAir:R6G6C-A01 -> Diodes_SMD:D_0603
- R1: value 1k -> 100; moved to F.Cu
- R3: value 100 -> 1k
- SW1: value POWER -> Push; footprint Buttons_Switches_SMD:SW_SPDT_PCM12 -> atreusAir:ASwitch; moved to F.Cu
- SW43: value Push -> POWER; footprint atreusAir:ASwitch -> Buttons_Switches_SMD:SW_SPDT_PCM12; moved to B.Cu
- U1: moved to B.Cu
- moved SW12 190.7 mm to (254.8, 92.5), turned to 0 degrees
- moved SW27 184.6 mm to (42.0, 54.5), turned to 0 degrees
- moved D12 182.6 mm to (253.3, 82.9), turned to 0 degrees
- moved D27 177.8 mm to (44.6, 45.5), turned to 0 degrees
- moved SW11 170.5 mm to (236.1, 89.4), turned to 0 degrees
- moved D11 163.1 mm to (237.4, 80.7), turned to 0 degrees
- moved D38 162.6 mm to (44.6, 27.4), turned to 0 degrees
- moved SW38 161.8 mm to (179.1, 38.5), turned to 0 degrees
- moved D26 154.4 mm to (62.5, 43.2), turned to 0 degrees
- moved SW33 147.8 mm to (118.1, 38.2), turned to 0 degrees
- moved SW25 143.4 mm to (79.9, 46.5), turned to 0 degrees
- moved D10 140.9 mm to (217.4, 75.5), turned to 0 degrees
- moved SW10 137.0 mm to (216.9, 84.3), turned to 0 degrees
- moved SW17 129.4 mm to (42.0, 73.5), turned to 0 degrees
- moved SW26 126.2 mm to (61.1, 51.5), turned to 0 degrees
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Connections:
- D1 pad 2: ROW0 -> ROW4
- D11 pad 2: ROW1 -> ROW0
- D12 pad 2: ROW2 -> ROW0
- D13 pad 2: ROW0 -> ROW1
- D15 pad 2: ROW2 -> ROW1
- D16 pad 2: ROW0 -> ROW1
- D18 pad 2: ROW2 -> ROW1
- D19 pad 2: ROW0 -> ROW1
- D2 pad 2: ROW1 -> ROW4
- D21 pad 2: ROW2 -> ROW1
- D22 pad 2: ROW0 -> ROW1
- D23 pad 2: ROW1 -> ROW2
- D25 pad 2: ROW4 -> ROW2
- D26 pad 2: ROW0 -> ROW2
- D27 pad 2: ROW1 -> ROW2
- D29 pad 2: ROW4 -> ROW2
- D3 pad 2: ROW2 -> ROW0
- D30 pad 2: ROW0 -> ROW2
- D31 pad 2: ROW1 -> ROW2
- D33 pad 2: ROW3 -> Net-(D33-Pad2)
- D38 pad 2: ROW4 -> ROW3
- D43 pad 2: Net-(D43-Pad2) -> ROW4
- D5 pad 2: ROW1 -> ROW0
- D6 pad 2: ROW2 -> ROW0
- D8 pad 2: ROW1 -> ROW0
- D9 pad 2: ROW2 -> ROW0
- R1 pad 1: Net-(R1-Pad1) -> Net-(D33-Pad1)
- R1 pad 2: GND -> LEDR
- R2 pad 1: Net-(D43-Pad1) -> Net-(D33-Pad2)
- R2 pad 2: LEDR -> LEDG
- R3 pad 1: Net-(D43-Pad2) -> Net-(R3-Pad1)
- R3 pad 2: LEDG -> GND
- SW1 pad 1: Net-(SW1-Pad1) -> Net-(D1-Pad1)
- SW1 pad 2: Net-(SW1-Pad2) -> COL1
- SW10 pad 1: Net-(D9-Pad1) -> Net-(D10-Pad1)
- SW10 pad 2: COL3 -> COL8
- SW11 pad 1: Net-(D10-Pad1) -> Net-(D11-Pad1)
- SW11 pad 2: COL4 -> COL9
- SW12 pad 1: Net-(D11-Pad1) -> Net-(D12-Pad1)
- SW12 pad 2: COL4 -> COL10
- SW13 pad 1: Net-(D12-Pad1) -> Net-(D13-Pad1)
- SW13 pad 2: COL4 -> COL1
- SW14 pad 1: Net-(D13-Pad1) -> Net-(D14-Pad1)
- SW14 pad 2: COL5 -> COL2
- SW15 pad 1: Net-(D14-Pad1) -> Net-(D15-Pad1)
- SW15 pad 2: COL5 -> COL3
- SW16 pad 1: Net-(D15-Pad1) -> Net-(D16-Pad1)
- SW16 pad 2: COL5 -> COL4
- SW17 pad 1: Net-(D16-Pad1) -> Net-(D17-Pad1)
- SW17 pad 2: COL6 -> COL5
- SW18 pad 1: Net-(D17-Pad1) -> Net-(D18-Pad1)
- SW19 pad 1: Net-(D18-Pad1) -> Net-(D19-Pad1)
- SW19 pad 2: COL6 -> COL7
- SW2 pad 1: Net-(D1-Pad1) -> Net-(D2-Pad1)
- SW2 pad 2: COL1 -> COL2
- SW20 pad 1: Net-(D19-Pad1) -> Net-(D20-Pad1)
- SW20 pad 2: COL7 -> COL8
- SW21 pad 1: Net-(D20-Pad1) -> Net-(D21-Pad1)
- SW21 pad 2: COL7 -> COL9
- SW22 pad 1: Net-(D21-Pad1) -> Net-(D22-Pad1)
- SW22 pad 2: COL7 -> COL10
- SW23 pad 1: Net-(D22-Pad1) -> Net-(D23-Pad1)
- SW23 pad 2: COL8 -> COL1
- SW24 pad 1: Net-(D23-Pad1) -> Net-(D24-Pad1)
- SW24 pad 2: COL8 -> COL2
- SW25 pad 1: Net-(D24-Pad1) -> Net-(D25-Pad1)
- SW25 pad 2: COL8 -> COL3
- SW26 pad 1: Net-(D25-Pad1) -> Net-(D26-Pad1)
- SW26 pad 2: COL1 -> COL4
- SW27 pad 1: Net-(D26-Pad1) -> Net-(D27-Pad1)
- SW27 pad 2: COL9 -> COL5
- SW28 pad 1: Net-(D27-Pad1) -> Net-(D28-Pad1)
- SW28 pad 2: COL9 -> COL6
- SW29 pad 1: Net-(D28-Pad1) -> Net-(D29-Pad1)
- SW29 pad 2: COL9 -> COL7
- SW3 pad 1: Net-(D2-Pad1) -> Net-(D3-Pad1)
- SW30 pad 1: Net-(D29-Pad1) -> Net-(D30-Pad1)
- SW30 pad 2: COL2 -> COL8
- SW31 pad 1: Net-(D30-Pad1) -> Net-(D31-Pad1)
- SW31 pad 2: COL10 -> COL9
- SW32 pad 1: Net-(D31-Pad1) -> Net-(D32-Pad1)
- SW33 pad 1: Net-(D32-Pad1) -> Net-(D34-Pad1)
- SW33 pad 2: COL10 -> COL1
- SW34 pad 1: Net-(D33-Pad1) -> Net-(D35-Pad1)
- SW34 pad 2: COL1 -> COL2
- SW35 pad 1: Net-(D34-Pad1) -> Net-(D36-Pad1)
- SW35 pad 2: COL2 -> COL3
- SW36 pad 1: Net-(D35-Pad1) -> Net-(D37-Pad1)
- SW36 pad 2: COL3 -> COL4
- SW37 pad 1: Net-(D36-Pad1) -> Net-(D38-Pad1)
- SW37 pad 2: COL4 -> COL5
- SW38 pad 1: Net-(D37-Pad1) -> Net-(D39-Pad1)
- SW38 pad 2: COL5 -> COL6
- SW39 pad 1: Net-(D38-Pad1) -> Net-(D40-Pad1)
- SW39 pad 2: COL6 -> COL7
- SW4 pad 1: Net-(D3-Pad1) -> Net-(D4-Pad1)
- SW4 pad 2: COL1 -> COL2
- SW40 pad 1: Net-(D39-Pad1) -> Net-(D41-Pad1)
- SW40 pad 2: COL7 -> COL8
- SW41 pad 1: Net-(D40-Pad1) -> Net-(D42-Pad1)
- SW41 pad 2: COL8 -> COL9
- SW42 pad 1: Net-(D41-Pad1) -> Net-(D43-Pad1)
- SW42 pad 2: COL9 -> COL10
- SW43 pad 1: Net-(D42-Pad1) -> (no net)
- SW43 pad 2: COL10 -> Net-(SW43-Pad2)
- SW5 pad 1: Net-(D4-Pad1) -> Net-(D5-Pad1)
- SW5 pad 2: COL2 -> COL3
- SW6 pad 1: Net-(D5-Pad1) -> Net-(D6-Pad1)
- SW6 pad 2: COL2 -> COL4
- SW7 pad 1: Net-(D6-Pad1) -> Net-(D7-Pad1)
- SW7 pad 2: COL2 -> COL5
- SW8 pad 1: Net-(D7-Pad1) -> Net-(D8-Pad1)
- SW8 pad 2: COL3 -> COL6
- SW9 pad 1: Net-(D8-Pad1) -> Net-(D9-Pad1)
- SW9 pad 2: COL3 -> COL7
- U1 pad 1: Net-(U1-Pad1) -> (no net)
- U1 pad 11: Net-(U1-Pad11) -> (no net)
- U1 pad 12: Net-(U1-Pad12) -> (no net)
- U1 pad 13: Net-(U1-Pad13) -> (no net)
- U1 pad 16: Net-(U1-Pad16) -> (no net)
- U1 pad 2: Net-(U1-Pad2) -> (no net)
- U1 pad 26: Net-(U1-Pad26) -> (no net)
- U1 pad 27: Net-(SW1-Pad2) -> Net-(SW43-Pad2)
- U1 pad 28: VLED -> (no net)
- U1 pad 29: Net-(U1-Pad29) -> (no net)
- U1 pad 3: Net-(U1-Pad3) -> (no net)
- U1 pad 30: Net-(U1-Pad30) -> (no net)
- U1 pad 31: Net-(U1-Pad31) -> (no net)
Routing:
- net ROW1: track 332.4 -> 0.00 mm, vias 6 -> 0
- net ROW2: track 299.7 -> 0.00 mm, vias 2 -> 0
- net ROW0: track 295.4 -> 0.00 mm, vias 2 -> 0
- net COL10: track 173.8 -> 0.00 mm
- net COL5: track 170.2 -> 0.00 mm
- net COL2: track 161.4 -> 0.00 mm
- net COL9: track 155.3 -> 0.00 mm
- net COL4: track 150.1 -> 0.00 mm
- net ROW4: track 140.9 -> 0.00 mm
- net COL8: track 139.8 -> 0.00 mm
- net COL3: track 138.1 -> 0.00 mm
- net ROW3: track 132.0 -> 0.00 mm
- net COL1: track 125.7 -> 0.00 mm
- net COL7: track 119.7 -> 0.00 mm
- net COL6: track 97.2 -> 0.00 mm
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- removed copper zone on B.Cu, net GND
Other:
- board outline removed

Commit message: ausrichtung feather korrigiert ! !
Parts:
- D1, D10, D11, D12, D13, D14, D15, D16, D17, D18, D19, D2, D20, D21, D22, D23, D24, D25, D26, D27, D28, D29, D3, D30, D31, D32, D4, D5, D6, D7, D8, D9: moved to B.Cu
- D33: renamed from D34; moved to B.Cu
- D34: renamed from D35; moved to B.Cu
- D35: renamed from D36; moved to B.Cu
- D36: renamed from D37; moved to B.Cu
- D37: renamed from D38; moved to B.Cu
- D38: renamed from D39; moved to B.Cu
- D39: renamed from D40; moved to B.Cu
- D40: renamed from D41; moved to B.Cu
- D41: renamed from D42; moved to B.Cu
- D42: renamed from D43; moved to B.Cu
- R2: renamed from R1; moved to B.Cu
- R3: renamed from R2; moved to B.Cu
- moved SW32 213.2 mm to (42.0, 54.5)
- moved SW7 213.2 mm to (255.0, 92.5)
- moved SW42 213.0 mm to (42.0, 35.5)
- moved SW22 213.0 mm to (42.0, 73.5)
- moved SW37 213.0 mm to (255.0, 35.5)
- moved SW17 213.0 mm to (255.0, 73.5)
- moved SW27 212.9 mm to (255.0, 54.5)
- moved SW12 212.8 mm to (42.0, 92.5)
- moved D22 205.5 mm to (50.5, 67.0), turned to 90 degrees
- moved D32 204.9 mm to (50.5, 48.0), turned to 90 degrees
- moved D42 204.1 mm to (50.5, 29.0), turned to 90 degrees
- moved D12 202.9 mm to (50.5, 86.0), turned to 90 degrees
- moved D27 201.9 mm to (246.5, 48.0), turned to 90 degrees
- moved D37 201.9 mm to (246.5, 29.0), turned to 90 degrees
- moved D17 199.0 mm to (246.5, 67.0), turned to 90 degrees
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- renumbered D33 to D43, R3 to R1
Connections:
- D10 pad 2: ROW0 -> ROW4
- D11 pad 2: ROW0 -> ROW4
- D12 pad 2: ROW0 -> ROW4
- D38 pad 2: ROW4 -> ROW0
- D39 pad 2: ROW4 -> ROW0
- D40 pad 2: ROW4 -> ROW0
- D41 pad 2: ROW4 -> ROW0
- D42 pad 2: ROW4 -> ROW0
- D8 pad 2: ROW0 -> ROW4
- D9 pad 2: ROW0 -> ROW4
- R2 pad 2: LEDR -> LEDG
- R3 pad 2: LEDG -> LEDR
- SW1 pad 2: COL1 -> COL6
- SW2 pad 2: COL2 -> COL1
- SW43 pad 1: (no net) -> Net-(SW43-Pad1)
- U1 pad 1: (no net) -> Net-(U1-Pad1)
- U1 pad 11: (no net) -> Net-(U1-Pad11)
- U1 pad 12: (no net) -> Net-(U1-Pad12)
- U1 pad 13: (no net) -> Net-(U1-Pad13)
- U1 pad 16: (no net) -> Net-(U1-Pad16)
- U1 pad 2: (no net) -> Net-(U1-Pad2)
- U1 pad 26: (no net) -> Net-(U1-Pad26)
- U1 pad 28: (no net) -> VLED
- U1 pad 29: (no net) -> Net-(U1-Pad29)
- U1 pad 3: (no net) -> Net-(U1-Pad3)
- U1 pad 30: (no net) -> Net-(U1-Pad30)
- U1 pad 31: (no net) -> Net-(U1-Pad31)
Routing:
- net ROW2: track 0.00 -> 195.9 mm
- net ROW1: track 0.00 -> 195.6 mm
- net ROW0: track 0.00 -> 167.7 mm
- net ROW4: track 0.00 -> 93.1 mm
- net ROW3: track 0.00 -> 84.0 mm
- net COL6: track 0.00 -> 80.4 mm
- net COL1: track 0.00 -> 79.2 mm
- net COL2: track 0.00 -> 60.4 mm
- net COL10: track 0.00 -> 60.4 mm
- net COL9: track 0.00 -> 60.3 mm
- net COL8: track 0.00 -> 60.1 mm
- net COL7: track 0.00 -> 60.0 mm
- net COL3: track 0.00 -> 59.7 mm
- net COL4: track 0.00 -> 59.6 mm
- net COL5: track 0.00 -> 59.5 mm
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
Commit message: feather jetzt auf unterseite, leiterbahnen verlegt.
Parts:
- moved D43 50.0 mm to (82.0, 24.0), turned to 0 degrees
- moved R3 46.6 mm to (87.0, 23.5), turned to 0 degrees
- moved R2 45.2 mm to (87.0, 25.0), turned to 0 degrees
- moved R1 28.2 mm to (99.9, 25.1)
- moved SW43 28.1 mm to (94.5, 24.0)
- moved U1 19.0 mm to (147.5, 68.0)
- moved D33 19.0 mm to (161.1, 48.5), turned to 100 degrees
- moved D2 18.7 mm to (153.1, 98.2), turned to 100 degrees
- moved D38 18.1 mm to (133.8, 48.5), turned to 80 degrees
- moved SW1 17.7 mm to (134.8, 103.6), turned to 350 degrees
- moved SW2 17.5 mm to (160.1, 103.5), turned to 10 degrees
- moved D23 17.3 mm to (164.4, 67.2), turned to 100 degrees
- moved SW33 17.2 mm to (170.6, 53.5), turned to 10 degrees
- moved D34 17.0 mm to (178.9, 40.3), turned to 100 degrees
- moved D28 16.7 mm to (130.5, 67.3), turned to 80 degrees
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Connections:
- R2 pad 2: LEDG -> LEDR
- R3 pad 2: LEDR -> LEDG
Routing:
- net COL5: track 59.5 -> 175.5 mm, vias 0 -> 2
- net COL10: track 60.4 -> 167.2 mm, vias 0 -> 2
- net ROW0: track 167.7 -> 258.8 mm, vias 0 -> 3
- net COL4: track 59.6 -> 141.3 mm, vias 0 -> 1
- net COL9: track 60.3 -> 135.7 mm, vias 0 -> 1
- net Net-(SW43-Pad2): track 6.92 -> 67.2 mm
- net COL8: track 60.1 -> 119.9 mm
- net LEDG: track 42.0 -> 101.6 mm, vias 0 -> 1
- net LEDR: track 38.9 -> 96.5 mm, vias 0 -> 1
- net COL3: track 59.7 -> 116.8 mm, vias 0 -> 2
- net ROW3: track 84.0 -> 125.8 mm, vias 0 -> 1
- net ROW4: track 93.1 -> 134.2 mm
- net COL2: track 60.4 -> 100.7 mm, vias 0 -> 1
- net COL7: track 60.0 -> 93.7 mm
- net ROW1: track 195.6 -> 220.9 mm
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- added copper zone on B.Cu, net GND
- added copper zone on F.Cu, net GND
Other:
- board outline added: 239 x 97 mm
