File: atreusAir.kicad_pcb (KiCad board)
At the start: 2 copper layers, 239 x 97 mm, 90 parts, among them SW1 Push, SW10 Push, SW11 Push, SW12 Push, SW13 Push, SW14 Push, SW15 Push, SW16 Push, SW17 Push, SW18 Push, SW19 Push, SW2 Push, SW20 Push, SW21 Push, SW22 Push, SW23 Push, SW24 Push, SW25 Push, SW26 Push, SW27 Push, SW28 Push, SW29 Push, SW3 Push, SW30 Push, SW31 Push, SW32 Push, SW33 Push, SW34 Push, SW35 Push, SW36 Push, SW37 Push, SW38 Push, SW39 Push, SW4 Push, SW40 Push, SW41 Push, SW42 Push, SW43 POWER, SW5 Push, SW6 Push, SW7 Push, SW8 Push, SW9 Push, U1 Feather_Bluefruit_LE

Commit message: cleanup
Parts:
- added REF**: MountingHole_3.2mm_M3_DIN965, Mounting_Holes:MountingHole_3.2mm_M3_DIN965, F.Cu at (57.0, 26.0)
- added REF**: MountingHole_3.2mm_M3_DIN965, Mounting_Holes:MountingHole_3.2mm_M3_DIN965, F.Cu at (238.0, 26.0)
- added REF**: MountingHole_3.2mm_M3_DIN965, Mounting_Holes:MountingHole_3.2mm_M3_DIN965, F.Cu at (220.0, 105.0)
- added REF**: MountingHole_3.2mm_M3_DIN965, Mounting_Holes:MountingHole_3.2mm_M3_DIN965, F.Cu at (75.0, 105.0)
Changed lines of the file:
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@@
     (area 27.924999 21.924999 267.075001 119.075001)
     (thickness 0.8)
-    (drawings 12)
+    (drawings 16)
     (tracks 487)
     (zones 0)
-    (modules 90)
+    (modules 94)
     (nets 78)
   )
@@
     (pad_drill 2)
     (pad_to_mask_clearance 0.2)
-    (aux_axis_origin 0 0)
+    (aux_axis_origin 27.94 119.38)
     (visible_elements FFFFFF7F)
     (pcbplotparams
-      (layerselection 0x01000_80000001)
+      (layerselection 0x010cc_80000001)
       (usegerberextensions false)
       (excludeedgelayer true)
@@
       (viasonmask false)
       (mode 1)
-      (useauxorigin false)
+      (useauxorigin true)
       (hpglpennumber 1)
       (hpglpenspeed 20)
@@
       (drillshape 0)
       (scaleselection 1)
-      (outputdirectory export2019-02-24/))
+      (outputdirectory ../export/gerber/))
   )
   (net 0 "")
@@
     (descr "Ultraminiature Surface Mount Slide Switch")
     (attr smd)
-    (fp_text reference SW43 (at 0 3.2) (layer B.SilkS)
+    (fp_text reference SW43 (at -2.5 3.5) (layer B.SilkS)
       (effects (font (size 1 1) (thickness 0.15)) (justify mirror))
     )
-    (fp_text value POWER (at 0 -4.25) (layer B.Fab)
+    (fp_text value POWER (at 3 3.5) (layer B.Fab)
       (effects (font (size 1 1) (thickness 0.15)) (justify mirror))
     )
-    (fp_text user %R (at 0 3.2) (layer B.Fab)
+    (fp_text user %R (at -2.5 3.5) (layer B.Fab)
       (effects (font (size 1 1) (thickness 0.15)) (justify mirror))
     )
@@
     (tags "resistor 0603")
     (attr smd)
-    (fp_text reference R3 (at 0 1.45) (layer B.SilkS)
+    (fp_text reference R3 (at 2 0) (layer B.SilkS)
       (effects (font (size 1 1) (thickness 0.15)) (justify mirror))
     )
-    (fp_text value 100 (at 0 -1.5) (layer B.Fab)
+    (fp_text value 100 (at -3 0) (layer B.Fab)
       (effects (font (size 1 1) (thickness 0.15)) (justify mirror))
     )
@@
     (tags "resistor 0603")
     (attr smd)
-    (fp_text reference R2 (at 0 1.45) (layer B.SilkS)
+    (fp_text reference R2 (at 2 0) (layer B.SilkS)
       (effects (font (size 1 1) (thickness 0.15)) (justify mirror))
     )
-    (fp_text value 100 (at 0 -1.5) (layer B.Fab)
+    (fp_text value 100 (at -3 0) (layer B.Fab)
       (effects (font (size 1 1) (thickness 0.15)) (justify mirror))
     )
@@
   (module atreusAir:R6G6C-A01 (layer F.Cu)
     (at 82 24)
-    (fp_text reference D43 (at 0 5.75) (layer F.SilkS)
+    (fp_text reference D43 (at 1 1) (layer F.SilkS)
       (effects (font (size 1 1) (thickness 0.15)))
     )
-    (fp_text value 18-225/R6G6C-A01/3T (at -0.25 -5) (layer F.Fab)
+    (fp_text value 18-225/R6G6C-A01/3T (at -0.25 -5) (layer F.Fab) hide
       (effects (font (size 1 1) (thickness 0.15)))
     )
@@
     )
   )
+  (module Mounting_Holes:MountingHole_3.2mm_M3_DIN965 (layer F.Cu)
+    (at 57 26)
+    (descr "Mounting Hole 3.2mm, no annular, M3, DIN965")
+    (tags "mounting hole 3.2mm no annular m3 din965")
+    (attr virtual)
+    (fp_text reference REF** (at 0 -3.8) (layer F.SilkS) hide
+      (effects (font (size 1 1) (thickness 0.15)))
+    )
+    (fp_text value MountingHole_3.2mm_M3_DIN965 (at 0 3.8) (layer F.Fab) hide
+      (effects (font (size 1 1) (thickness 0.15)))
+    )
+    (fp_text user %R (at 0.3 0) (layer F.Fab)
+      (effects (font (size 1 1) (thickness 0.15)))
+    )
+    (fp_circle (center 0 0) (end 2.8 0) (layer Cmts.User) (width 0.15))
+    (fp_circle (center 0 0) (end 3.05 0) (layer F.CrtYd) (width 0.05))
+    (pad 1 np_thru_hole circle (at 0 0) (size 3.2 3.2) (drill 3.2) (layers *.Cu *.Mask))
+  )
+  (module Mounting_Holes:MountingHole_3.2mm_M3_DIN965 (layer F.Cu)
+    (at 238 26)
+    (descr "Mounting Hole 3.2mm, no annular, M3, DIN965")
+    (tags "mounting hole 3.2mm no annular m3 din965")
+    (attr virtual)
+    (fp_text reference REF** (at 0 -3.8) (layer F.SilkS) hide
+      (effects (font (size 1 1) (thickness 0.15)))
+    )
+    (fp_text value MountingHole_3.2mm_M3_DIN965 (at 0 3.8) (layer F.Fab) hide
+      (effects (font (size 1 1) (thickness 0.15)))
+    )
+    (fp_text user %R (at 0.3 0) (layer F.Fab)
+      (effects (font (size 1 1) (thickness 0.15)))
+    )
+    (fp_circle (center 0 0) (end 2.8 0) (layer Cmts.User) (width 0.15))
+    (fp_circle (center 0 0) (end 3.05 0) (layer F.CrtYd) (width 0.05))
+    (pad 1 np_thru_hole circle (at 0 0) (size 3.2 3.2) (drill 3.2) (layers *.Cu *.Mask))
+  )
+  (module Mounting_Holes:MountingHole_3.2mm_M3_DIN965 (layer F.Cu)
+    (at 220 105)
+    (descr "Mounting Hole 3.2mm, no annular, M3, DIN965")
+    (tags "mounting hole 3.2mm no annular m3 din965")
+    (attr virtual)
+    (fp_text reference REF** (at 0 -3.8) (layer F.SilkS) hide
+      (effects (font (size 1 1) (thickness 0.15)))
+    )
+    (fp_text value MountingHole_3.2mm_M3_DIN965 (at 0 3.8) (layer F.Fab) hide
+      (effects (font (size 1 1) (thickness 0.15)))
+    )
+    (fp_text user %R (at 0.3 0) (layer F.Fab)
+      (effects (font (size 1 1) (thickness 0.15)))
+    )
+    (fp_circle (center 0 0) (end 2.8 0) (layer Cmts.User) (width 0.15))
+    (fp_circle (center 0 0) (end 3.05 0) (layer F.CrtYd) (width 0.05))
+    (pad 1 np_thru_hole circle (at 0 0) (size 3.2 3.2) (drill 3.2) (layers *.Cu *.Mask))
+  )
+  (module Mounting_Holes:MountingHole_3.2mm_M3_DIN965 (layer F.Cu)
+    (at 75 105)
+    (descr "Mounting Hole 3.2mm, no annular, M3, DIN965")
+    (tags "mounting hole 3.2mm no annular m3 din965")
+    (attr virtual)
+    (fp_text reference REF** (at 0 -3.8) (layer F.SilkS) hide
+      (effects (font (size 1 1) (thickness 0.15)))
+    )
+    (fp_text value MountingHole_3.2mm_M3_DIN965 (at 0 3.8) (layer F.Fab) hide
+      (effects (font (size 1 1) (thickness 0.15)))
+    )
+    (fp_text user %R (at 0.3 0) (layer F.Fab)
+      (effects (font (size 1 1) (thickness 0.15)))
+    )
+    (fp_circle (center 0 0) (end 2.8 0) (layer Cmts.User) (width 0.15))
+    (fp_circle (center 0 0) (end 3.05 0) (layer F.CrtYd) (width 0.05))
+    (pad 1 np_thru_hole circle (at 0 0) (size 3.2 3.2) (drill 3.2) (layers *.Cu *.Mask))
+  )
+  (dimension 97 (width 0.3) (layer Cmts.User)
+    (gr_text "97,000 mm" (at -2.35 70.5 90) (layer Cmts.User)
+      (effects (font (size 1.5 1.5) (thickness 0.3)))
+    )
+    (feature1 (pts (xy 118 22) (xy -3.7 22)))
+    (feature2 (pts (xy 118 119) (xy -3.7 119)))
+    (crossbar (pts (xy -1 119) (xy -1 22)))
+    (arrow1a (pts (xy -1 22) (xy -0.413579 23.126504)))
+    (arrow1b (pts (xy -1 22) (xy -1.586421 23.126504)))
+    (arrow2a (pts (xy -1 119) (xy -0.413579 117.873496)))
+    (arrow2b (pts (xy -1 119) (xy -1.586421 117.873496)))
+  )
+  (dimension 239 (width 0.3) (layer Cmts.User)
+    (gr_text "239,000 mm" (at 147.5 136.35) (layer Cmts.User)
+      (effects (font (size 1.5 1.5) (thickness 0.3)))
+    )
+    (feature1 (pts (xy 28 98) (xy 28 137.7)))
+    (feature2 (pts (xy 267 98) (xy 267 137.7)))
+    (crossbar (pts (xy 267 135) (xy 28 135)))
+    (arrow1a (pts (xy 28 135) (xy 29.126504 134.413579)))
+    (arrow1b (pts (xy 28 135) (xy 29.126504 135.586421)))
+    (arrow2a (pts (xy 267 135) (xy 265.873496 134.413579)))
+    (arrow2b (pts (xy 267 135) (xy 265.873496 135.586421)))
+  )
+  (target plus (at 147.32 121.92) (size 5) (width 0.15) (layer Edge.Cuts))
+  (target plus (at 147.32 20.32) (size 5) (width 0.15) (layer Edge.Cuts))
   (gr_line (start 265 101.5) (end 267 98) (angle 90) (layer Edge.Cuts) (width 0.15))
   (gr_line (start 176 119) (end 265 101.5) (angle 90) (layer Edge.Cuts) (width 0.15))
